File: BurnWireControl.kicad_sch (KiCad schematic)
At the start: 37 parts, among them J10 Conn_01x02, J7 Conn_01x02, J8 Conn_01x02, J9 Conn_01x02, K1 9-1462038-9, Q1 MMBT2222AT, Q2 IRLML2803, Q3 IRLML2803, Q4 IRLML2803, Q5 IRLML2803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

Commit message: Finish v1 schematic
Parts:
- K1: footprint 914620389 -> (none)
- Q1: footprint mainboard:SOT-23 -> (none)
- Q6, Q7, Q8, Q9: footprint mainboard:NDS8434 -> (none)
Changed lines of the file:
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@@
 			)
 		)
-		(property "Footprint" "mainboard:NDS8434"
+		(property "Footprint" ""
 			(at 208.28 101.6 0)
 			(effects
@@
 			)
 		)
-		(property "Footprint" "914620389"
+		(property "Footprint" ""
 			(at 105.41 92.71 0)
 			(effects
@@
 			)
 		)
-		(property "Footprint" "mainboard:NDS8434"
+		(property "Footprint" ""
 			(at 208.28 127 0)
 			(effects
@@
 			)
 		)
-		(property "Footprint" "mainboard:SOT-23"
+		(property "Footprint" ""
 			(at 52.07 102.87 0)
 			(effects
@@
 			)
 		)
-		(property "Footprint" "mainboard:NDS8434"
+		(property "Footprint" ""
 			(at 208.28 50.8 0)
 			(effects
@@
 			)
 		)
-		(property "Footprint" "mainboard:NDS8434"
+		(property "Footprint" ""
 			(at 208.28 76.2 0)
 			(effects
