File: BatteryProtection.kicad_sch (KiCad schematic)
At the start: 54 parts, among them Q10 Si7625DN, Q11 Si7625DN, Q12 Si7625DN, Q13 Si7625DN, U1 S-8209AAA-T8T1U, U2 MAX17205, U3 S-8209AAA-T8T1U, U4 LTC4412xS6, U5 LTC4412xS6

Commit message: Finish v1 schematic
Parts:
- C1, C10, C11, C2, C3, C4, C5, C6, C7, C8, C9: footprint (none) -> Capacitor_SMD:C_0603_1608Metric
- R18, R19, R20, R21, R22, R23, R24, R26, R27, R28, R29, R30: footprint (none) -> Resistor_SMD:R_0603_1608Metric
- R25: footprint (none) -> Resistor_SMD:R_2512_6332Metric
- U1, U3: footprint (none) -> Package_SO:TSSOP-8_4.4x3mm_P0.65mm
- U2: footprint (none) -> Package_DFN_QFN:TDFN-14-1EP_3x3mm_P0.4mm_EP1.78x2.35mm
Connections:
- net GND: now also U2.15 (GND)
Other:
- moved on the sheet: C10, C8, TP14

Commit message: Cleanup component designators
Parts:
- removed TP1, TP2, TP3: TestPoint, TestPoint:TestPoint_Loop_D1.80mm_Drill1.0mm_Beaded, symbol Connector:TestPoint
- renumbered Q10 to Q1, Q12 to Q2, Q11 to Q3, Q13 to Q4, R25 to R13, R20 to R14, R21 to R15, R27 to R16, R28 to R17, R22 to R20, R23 to R21, R24 to R22, R26 to R23, R30 to R24, R29 to R25, TP4 to TP1, TP6 to TP10, TP8 to TP11, TP9 to TP12, TP7 to TP13, TP10 to TP14, TP5 to TP2, TP11 to TP3, TP12 to TP4, TP15 to TP5, TP13 to TP6, TP14 to TP7, TP17 to TP8, TP18 to TP9, U3 to U1, U1 to U2, U2 to U3
Connections:
- net Alert_Fuel renamed ALRT
Other:
- moved on the sheet: TP11

Commit message: Complete layout
Parts:
- F1, F2: footprint (none) -> Resistor_SMD:R_1206_3216Metric
- TP1, TP10, TP11, TP12, TP13, TP14, TP2, TP3, TP4, TP5, TP6, TP7, TP8, TP9: footprint TestPoint:TestPoint_Loop_D1.80mm_Drill1.0mm_Beaded -> TestPoint:TestPoint_THTPad_D1.0mm_Drill0.5mm
Connections:
- net CHRG_STAT renamed CSTAT
- net DCHRG_STAT renamed DSTAT
Other:
- note added: "1206 3A"
- note added: "1206 6A"
- moved on the sheet: TP6, TP8
Changed lines of the file:
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@@
 	(wire
 		(pts
+			(xy 194.31 64.77) (xy 201.93 64.77)
+		)
+		(stroke
+			(width 0)
+			(type default)
+		)
+	)
+	(wire
+		(pts
 			(xy 199.39 133.35) (xy 212.09 133.35)
 		)
@@
 	(wire
 		(pts
-			(xy 222.25 123.19) (xy 236.22 123.19)
+			(xy 222.25 123.19) (xy 229.87 123.19)
 		)
 		(stroke
@@
 	(wire
 		(pts
-			(xy 190.5 64.77) (xy 201.93 64.77)
-		)
-		(stroke
-			(width 0)
-			(type default)
-		)
-	)
-	(wire
-		(pts
 			(xy 31.75 115.57) (xy 43.18 115.57)
 		)
@@
 		)
 	)
+	(text "1206 6A"
+		(exclude_from_sim no)
+		(at 163.83 89.154 0)
+		(effects
+			(font
+				(size 1.27 1.27)
+			)
+		)
+	)
 	(text "Battery protection design derived from \nPortland State University's \nOpen-Source OreSat project"
 		(exclude_from_sim no)
@@
 		)
 	)
+	(text "1206 3A"
+		(exclude_from_sim no)
+		(at 163.576 36.83 0)
+		(effects
+			(font
+				(size 1.27 1.27)
+			)
+		)
+	)
 	(text "t_D = 10.0 MΩ typ. × C_CDT [μF]\nt_D = 0.1s"
 		(exclude_from_sim no)
@@
 		)
 	)
-	(label "CHRG_STAT"
-		(at 190.5 64.77 0)
-		(fields_autoplaced yes)
-		(effects
-			(font
-				(size 1.27 1.27)
-			)
-			(justify left bottom)
-		)
-	)
-	(label "DCHRG_STAT"
-		(at 236.22 123.19 180)
-		(fields_autoplaced yes)
-		(effects
-			(font
-				(size 1.27 1.27)
-			)
-			(justify right bottom)
-		)
-	)
 	(global_label "B-"
 		(shape bidirectional)
@@
 		)
 	)
+	(global_label "CSTAT"
+		(shape bidirectional)
+		(at 194.31 64.77 180)
+		(fields_autoplaced yes)
+		(effects
+			(font
+				(size 1.27 1.27)
+			)
+			(justify right)
+		)
+		(property "Intersheetrefs" "${INTERSHEET_REFS}"
+			(at 185.5232 64.77 0)
+			(effects
+				(font
+					(size 1.27 1.27)
+				)
+				(justify right)
+				(hide yes)
+			)
+		)
+	)
 	(global_label "ALRT"
 		(shape bidirectional)
@@
 		)
 	)
+	(global_label "DSTAT"
+		(shape bidirectional)
+		(at 229.87 123.19 270)
+		(fields_autoplaced yes)
+		(effects
+			(font
+				(size 1.27 1.27)
+			)
+			(justify right)
+		)
+		(property "Intersheetrefs" "${INTERSHEET_REFS}"
+			(at 229.87 131.9768 90)
+			(effects
+				(font
+					(size 1.27 1.27)
+				)
+				(justify right)
+				(hide yes)
+			)
+		)
+	)
 	(global_label "B+"
 		(shape bidirectional)
@@
 		(dnp no)
 		(property "Reference" "F1"
-			(at 163.83 28.448 90)
+			(at 163.83 30.48 90)
 			(effects
 				(font
@@
 		)
 		(property "Value" "Polyfuse_Small"
-			(at 163.83 30.734 90)
+			(at 163.83 32.004 90)
 			(effects
 				(font
@@
 			)
 		)
-		(property "Footprint" ""
+		(property "Footprint" "Resistor_SMD:R_1206_3216Metric"
 			(at 168.91 33.02 0)
 			(effects
@@
 			)
 		)
-		(property "Footprint" "TestPoint:TestPoint_Loop_D1.80mm_Drill1.0mm_Beaded"
+		(property "Footprint" "TestPoint:TestPoint_THTPad_D1.0mm_Drill0.5mm"
 			(at 147.32 154.94 0)
 			(effects
@@
 			)
 		)
-		(property "Footprint" "TestPoint:TestPoint_Loop_D1.80mm_Drill1.0mm_Beaded"
+		(property "Footprint" "TestPoint:TestPoint_THTPad_D1.0mm_Drill0.5mm"
 			(at 154.94 160.02 0)
 			(effects
@@
 			)
 		)
-		(property "Footprint" "TestPoint:TestPoint_Loop_D1.80mm_Drill1.0mm_Beaded"
+		(property "Footprint" "TestPoint:TestPoint_THTPad_D1.0mm_Drill0.5mm"
 			(at 154.94 144.78 0)
 			(effects
@@
 			)
 		)
-		(property "Footprint" "TestPoint:TestPoint_Loop_D1.80mm_Drill1.0mm_Beaded"
+		(property "Footprint" "TestPoint:TestPoint_THTPad_D1.0mm_Drill0.5mm"
 			(at 152.4 59.69 0)
 			(effects
@@
 			)
 		)
-		(property "Footprint" "TestPoint:TestPoint_Loop_D1.80mm_Drill1.0mm_Beaded"
+		(property "Footprint" "TestPoint:TestPoint_THTPad_D1.0mm_Drill0.5mm"
 			(at 97.79 59.69 0)
 			(effects
@@
 	(symbol
 		(lib_id "Connector:TestPoint")
-		(at 236.22 123.19 270)
-		(mirror x)
+		(at 229.87 123.19 0)
+		(mirror y)
 		(unit 1)
 		(exclude_from_sim no)
@@
 		(dnp no)
 		(property "Reference" "TP8"
-			(at 243.078 123.19 90)
+			(at 232.664 119.888 0)
 			(effects
 				(font
@@
 		)
 		(property "Value" "TestPoint"
-			(at 236.9058 121.7168 0)
+			(at 228.3968 122.5042 0)
 			(effects
 				(font
@@
 			)
 		)
-		(property "Footprint" "TestPoint:TestPoint_Loop_D1.80mm_Drill1.0mm_Beaded"
-			(at 236.22 118.11 0)
+		(property "Footprint" "TestPoint:TestPoint_THTPad_D1.0mm_Drill0.5mm"
+			(at 224.79 123.19 0)
 			(effects
 				(font
@@
 		)
 		(property "Datasheet" "~"
-			(at 236.22 118.11 0)
+			(at 224.79 123.19 0)
 			(effects
 				(font
@@
 		)
 		(property "Description" ""
-			(at 236.22 123.19 0)
+			(at 229.87 123.19 0)
 			(effects
 				(font
@@
 		)
 		(property "DNP" "DNP"
-			(at 236.22 123.19 0)
+			(at 229.87 123.19 0)
 			(effects
 				(font
@@
 			)
 		)
-		(property "Footprint" "TestPoint:TestPoint_Loop_D1.80mm_Drill1.0mm_Beaded"
+		(property "Footprint" "TestPoint:TestPoint_THTPad_D1.0mm_Drill0.5mm"
 			(at 256.54 34.29 0)
 			(effects
@@
 			)
 		)
-		(property "Footprint" "TestPoint:TestPoint_Loop_D1.80mm_Drill1.0mm_Beaded"
+		(property "Footprint" "TestPoint:TestPoint_THTPad_D1.0mm_Drill0.5mm"
 			(at 189.23 91.44 0)
 			(effects
@@
 	(symbol
 		(lib_id "Connector:TestPoint")
-		(at 190.5 64.77 90)
-		(mirror x)
+		(at 194.31 64.77 0)
+		(mirror y)
 		(unit 1)
 		(exclude_from_sim no)
@@
 		(dnp no)
 		(property "Reference" "TP6"
-			(at 188.722 67.056 90)
+			(at 191.516 61.468 0)
 			(effects
 				(font
@@
 		)
 		(property "Value" "TestPoint"
-			(at 189.8142 66.2432 0)
+			(at 192.8368 64.0842 0)
 			(effects
 				(font
@@
 			)
 		)
-		(property "Footprint" "TestPoint:TestPoint_Loop_D1.80mm_Drill1.0mm_Beaded"
-			(at 190.5 69.85 0)
+		(property "Footprint" "TestPoint:TestPoint_THTPad_D1.0mm_Drill0.5mm"
+			(at 189.23 64.77 0)
 			(effects
 				(font
@@
 		)
 		(property "Datasheet" "~"
-			(at 190.5 69.85 0)
+			(at 189.23 64.77 0)
 			(effects
 				(font
@@
 		)
 		(property "Description" ""
-			(at 190.5 64.77 0)
+			(at 194.31 64.77 0)
 			(effects
 				(font
@@
 		)
 		(property "DNP" "DNP"
-			(at 190.5 64.77 0)
+			(at 194.31 64.77 0)
 			(effects
 				(font
@@
 			)
 		)
-		(property "Footprint" "TestPoint:TestPoint_Loop_D1.80mm_Drill1.0mm_Beaded"
+		(property "Footprint" "TestPoint:TestPoint_THTPad_D1.0mm_Drill0.5mm"
 			(at 127 115.57 0)
 			(effects
@@
 			)
 		)
-		(property "Footprint" "TestPoint:TestPoint_Loop_D1.80mm_Drill1.0mm_Beaded"
+		(property "Footprint" "TestPoint:TestPoint_THTPad_D1.0mm_Drill0.5mm"
 			(at 93.98 54.61 0)
 			(effects
@@
 			)
 		)
-		(property "Footprint" "TestPoint:TestPoint_Loop_D1.80mm_Drill1.0mm_Beaded"
+		(property "Footprint" "TestPoint:TestPoint_THTPad_D1.0mm_Drill0.5mm"
 			(at 194.31 34.29 0)
 			(effects
@@
 		(dnp no)
 		(property "Reference" "F2"
-			(at 163.83 97.282 90)
+			(at 163.83 96.012 90)
 			(effects
 				(font
@@
 		)
 		(property "Value" "Polyfuse_Small"
-			(at 163.83 94.996 90)
+			(at 163.83 93.726 90)
 			(effects
 				(font
@@
 			)
 		)
-		(property "Footprint" ""
+		(property "Footprint" "Resistor_SMD:R_1206_3216Metric"
 			(at 168.91 90.17 0)
 			(effects
@@
 			)
 		)
-		(property "Footprint" "TestPoint:TestPoint_Loop_D1.80mm_Drill1.0mm_Beaded"
+		(property "Footprint" "TestPoint:TestPoint_THTPad_D1.0mm_Drill0.5mm"
 			(at 152.4 64.77 0)
 			(effects
@@
 			)
 		)
-		(property "Footprint" "TestPoint:TestPoint_Loop_D1.80mm_Drill1.0mm_Beaded"
+		(property "Footprint" "TestPoint:TestPoint_THTPad_D1.0mm_Drill0.5mm"
 			(at 144.78 144.78 0)
 			(effects
