File: BatteryBoard.kicad_pcb (KiCad board)
At the start: 2 copper layers, 95.9 x 90.2 mm, 71 parts, among them IC2 BQ29209TDRBTQ1, IC3 PJA3412-AU_R1_000A1, J1 1042, J10 2383942-2, J11 2383942-2, J12 686114148922, J13 2383942-2, J14 2383942-2, J15 2383942-2, J2 1042, J3 1042, J4 1042, J5 1042, J6 1042, J7 2383942-2, J8 2383942-2, J9 2383942-2, K1 9-1462038-9, Q10 IRLML2803, Q11 IRLML2803, Q3 MMBT2222AT, Q4 IRLML2803, Q5 IRLML2803, Q6 NDS8434, Q7 NDS8434, Q8 NDS8434, Q9 NDS8434

Commit message: Finish v1 schematic
Parts:
- removed D2: DFLS130L-7, SamacSys_Parts:POWERDI_123
- removed G*** (x2): LOGO, Symbol:Argus LOGO 10x6.4
- removed IC2: BQ29209TDRBTQ1, SamacSys_Parts:SON65P300X300X100-9N-D
- removed IC3: PJA3412-AU_R1_000A1, SamacSys_Parts:SOT95P240X110-3N
- removed J10, J13, J15, J7, J8, J9: 2383942-2, SamacSys_Parts:23839422
- removed J12: 686114148922, SamacSys_Parts:686114148922
- removed K1: 9-1462038-9, SamacSys_Parts:914620389
- removed Q3: MMBT2222AT, mainboard:SOT-23
- removed Q4, Q5: IRLML2803, mainboard:SOT-23
- removed Q6, Q7, Q8, Q9: NDS8434, mainboard:NDS8434
- removed R10, R11, R12, R13: 100k, Resistor_SMD:R_0603_1608Metric
- removed R14, R15, R8, R9: 4.7k, Resistor_SMD:R_0603_1608Metric
- removed R16, R17, R5, R6, R7: 10k, Resistor_SMD:R_0603_1608Metric
- removed RV1: ITV4030L0812NR, SamacSys_Parts:ITV4030L0812NR
- added C10: 0.1uF, Capacitor_SMD:C_0603_1608Metric, F.Cu at (202.8, 139.0)
- added C11: 0.1uF, Capacitor_SMD:C_0603_1608Metric, F.Cu at (191.7, 124.2)
- added C12: 10nF, Capacitor_SMD:C_0603_1608Metric, B.Cu at (194.2, 88.7)
- added C13: 10nF, Capacitor_SMD:C_0603_1608Metric, B.Cu at (198.9, 88.7)
- added C4: 1nF, Capacitor_SMD:C_0603_1608Metric, B.Cu at (225.1, 88.2)
- added C5: 0.1uF, Capacitor_SMD:C_0603_1608Metric, B.Cu at (230.1, 89.7)
- added C6: 0.1uF, Capacitor_SMD:C_0603_1608Metric, F.Cu at (189.0, 120.6)
- added C7: 10nF, Capacitor_SMD:C_0603_1608Metric, F.Cu at (191.3, 121.3)
- added C9: 0.47uF, Capacitor_SMD:C_0603_1608Metric, B.Cu at (220.1, 85.8)
- added Q12: Si7625DN, Package_SO:Vishay_PowerPAK_1212-8_Single, F.Cu at (195.0, 130.0)
- added Q13: Si7625DN, Package_SO:Vishay_PowerPAK_1212-8_Single, F.Cu at (205.7, 140.8)
- added Q14: NX3008NBKS, Package_TO_SOT_SMD:SOT-363_SC-70-6, B.Cu at (194.2, 86.8)
- added Q15: MBT2222ADW1T1, Package_TO_SOT_SMD:SOT-363_SC-70-6, B.Cu at (194.2, 82.8)
- added Q16: NX3008NBKS, Package_TO_SOT_SMD:SOT-363_SC-70-6, B.Cu at (198.9, 86.7)
- added Q17: MBT2222ADW1T1, Package_TO_SOT_SMD:SOT-363_SC-70-6, B.Cu at (198.9, 82.8)
- added R24: 1K, Resistor_SMD:R_0603_1608Metric, F.Cu at (188.3, 118.4)
- added R25: 10m, Resistor_SMD:R_2512_6332Metric, B.Cu at (222.3, 81.8)
- added R26: 470R, Resistor_SMD:R_0603_1608Metric, F.Cu at (187.6, 120.6)
- added R27: 10K, Resistor_SMD:R_0603_1608Metric, B.Cu at (222.3, 90.5)
- added R28: 10K, Resistor_SMD:R_0603_1608Metric, B.Cu at (222.3, 92.0)
- added R29: 100K, Resistor_SMD:R_0603_1608Metric, F.Cu at (208.6, 137.0)
- added R30: 100K, Resistor_SMD:R_0603_1608Metric, F.Cu at (197.5, 127.8)
- added R31: 680R, Resistor_SMD:R_0603_1608Metric, B.Cu at (194.2, 80.8)
- added R32: 100K, Resistor_SMD:R_0603_1608Metric, B.Cu at (191.9, 87.7)
- added R33: 10K, Resistor_SMD:R_0603_1608Metric, B.Cu at (194.2, 79.4)
- added R34: 10K, Resistor_SMD:R_0603_1608Metric, B.Cu at (191.9, 84.7)
- added R35: 200K, Resistor_SMD:R_0603_1608Metric, B.Cu at (194.2, 84.8)
- added R36: 680R, Resistor_SMD:R_0603_1608Metric, B.Cu at (198.9, 80.8)
- added R37: 100K, Resistor_SMD:R_0603_1608Metric, B.Cu at (196.6, 87.7)
- added R38: 10K, Resistor_SMD:R_0603_1608Metric, B.Cu at (198.9, 79.3)
- added R39: 10K, Resistor_SMD:R_0603_1608Metric, B.Cu at (196.6, 84.7)
- added R40: 200K, Resistor_SMD:R_0603_1608Metric, B.Cu at (198.9, 84.8)
- added R41: DNI (0R), Resistor_SMD:R_0603_1608Metric, B.Cu at (191.9, 81.8)
- added R42: DNI (0R), Resistor_SMD:R_0603_1608Metric, B.Cu at (196.6, 81.7)
- added TH2: 197-103LAG-A01, Resistor_THT:R_Axial_DIN0204_L3.6mm_D1.6mm_P5.08mm_Vertical, F.Cu at (246.3, 160.9)
- added TP13: TestPoint, TestPoint:TestPoint_Loop_D1.80mm_Drill1.0mm_Beaded, F.Cu at (264.3, 120.5)
- added TP14: TestPoint, TestPoint:TestPoint_Loop_D1.80mm_Drill1.0mm_Beaded, F.Cu at (264.3, 125.1)
- added TP15: TestPoint, TestPoint:TestPoint_Loop_D1.80mm_Drill1.0mm_Beaded, F.Cu at (264.3, 129.8)
- added TP17: TestPoint, TestPoint:TestPoint_Loop_D1.80mm_Drill1.0mm_Beaded, F.Cu at (264.3, 134.4)
- added TP18: TestPoint, TestPoint:TestPoint_Loop_D1.80mm_Drill1.0mm_Beaded, F.Cu at (264.3, 139.1)
- added TP19: TestPoint, TestPoint:TestPoint_Loop_D1.80mm_Drill1.0mm_Beaded, F.Cu at (271.6, 136.9)
- added TP24: TestPoint, TestPoint:TestPoint_Loop_D1.80mm_Drill1.0mm_Beaded, F.Cu at (271.6, 141.6)
- added U1: S-8209AAA-T8T1U, Package_SO:TSSOP-8_4.4x3mm_P0.65mm, F.Cu at (181.3, 118.9)
- added U2: MAX17205, Package_DFN_QFN:TDFN-14-1EP_3x3mm_P0.4mm_EP1.78x2.35mm, B.Cu at (222.6, 86.4)
- added U3: S-8209AAA-T8T1U, Package_SO:TSSOP-8_4.4x3mm_P0.65mm, F.Cu at (193.7, 118.8)
- added U4: LTC4412xS6, Package_TO_SOT_SMD:TSOT-23-6, F.Cu at (191.5, 127.0)
- added U5: LTC4412xS6, Package_TO_SOT_SMD:TSOT-23-6, F.Cu at (209.6, 140.6)
- C1: value C0805C104K8JACAUTO -> 0.1uF; footprint SamacSys_Parts:CAPC2012X88N -> Capacitor_SMD:C_0603_1608Metric; moved to F.Cu
- C2: value C0805C104K8JACAUTO -> 10nF; footprint SamacSys_Parts:CAPC2012X88N -> Capacitor_SMD:C_0603_1608Metric; moved to F.Cu
- C3: value C0805C104K8JACAUTO -> 1nF; footprint SamacSys_Parts:CAPC2012X88N -> Capacitor_SMD:C_0603_1608Metric
- C8: value C0805C334K5RACAUTO -> 0.47uF; footprint SamacSys_Parts:C0805 -> Capacitor_SMD:C_0603_1608Metric
- H1, H2: footprint custom-footprints:MountingHole_3.2mm_M3_DIN965_PadMOD -> BatteryBoard:MountingHole; moved to F.Cu
- H3, H4: footprint custom-footprints:MountingHole_3.2mm_M3_DIN965_PadMOD -> BatteryBoard:MountingHole
- J1, J3, J6: value 1042 -> Keystone-1042; footprint SamacSys_Parts:KEYSTONE-1042 -> BatteryBoard:Keystone_1042
- J11: value 2383942-2 -> 200528-0120; footprint SamacSys_Parts:23839422 -> Connector_FFC-FPC:Molex_200528-0120_1x12-1MP_P1.00mm_Horizontal; moved to F.Cu
- J14: value 2383942-2 -> XT30PW; footprint SamacSys_Parts:23839422 -> BatteryBoard:AMASS_XT30PW-M; moved to F.Cu
- J2, J4: value 1042 -> Keystone-1042; footprint SamacSys_Parts:KEYSTONE-1042 -> BatteryBoard:Keystone_1042; moved to B.Cu
- J5: value 1042 -> Keystone-1042; footprint SamacSys_Parts:KEYSTONE-1042 -> BatteryBoard:Keystone_1042; moved to F.Cu
- Q10, Q11: value IRLML2803 -> Si7625DN; footprint mainboard:SOT-23 -> Package_SO:Vishay_PowerPAK_1212-8_Single; moved to F.Cu
- R18, R19: value ERJ-P06J271V -> 1K; footprint SamacSys_Parts:ERJP06D1000V -> Resistor_SMD:R_0603_1608Metric; moved to F.Cu
- R20: value ERJ-P06J221V -> 10R; footprint SamacSys_Parts:ERJP06D1000V -> Resistor_SMD:R_0603_1608Metric
- R21: value ERJ-P06J221V -> 100R; footprint SamacSys_Parts:ERJP06D1000V -> Resistor_SMD:R_0603_1608Metric
- R22: value ERJ-P06J102V -> 470R; footprint SamacSys_Parts:ERJP06D1000V -> Resistor_SMD:R_0603_1608Metric; moved to F.Cu
- R23: value ESR10EZPJ101 -> 1K; footprint SamacSys_Parts:RESC2012X65N -> Resistor_SMD:R_0603_1608Metric; moved to F.Cu
- TH1: value Thermistor -> 197-103LAG-A01; moved to F.Cu
- TP1, TP10, TP11, TP12, TP2, TP3, TP4, TP5, TP6, TP7, TP8, TP9: moved to F.Cu
- moved TP1 196.6 mm to (255.0, 120.5), turned to 0 degrees
- moved TP4 185.2 mm to (255.0, 134.4), turned to 0 degrees
- moved TP3 179.4 mm to (255.0, 129.8), turned to 0 degrees
- moved TP5 169.9 mm to (255.0, 139.1), turned to 0 degrees
- moved TH1 160.9 mm to (246.3, 157.8), turned to 0 degrees
- moved C3 157.2 mm to (225.1, 85.2), turned to -90 degrees
- moved C8 151.9 mm to (223.0, 79.1)
- moved R21 151.2 mm to (228.0, 89.2)
- moved TP6 148.9 mm to (255.0, 143.7), turned to 0 degrees
- moved R20 145.4 mm to (226.6, 85.3), turned to -90 degrees
- moved TP11 139.4 mm to (259.6, 139.1), turned to 0 degrees
- moved J11 135.9 mm to (216.4, 55.3)
- moved TP10 135.9 mm to (259.6, 134.4), turned to 0 degrees
- moved TP12 133.2 mm to (259.6, 143.7), turned to 0 degrees
- moved TP9 133.0 mm to (259.6, 129.8), turned to 0 degrees
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Connections:
- C1 pad 1: Net-(IC2-VC1) -> Net-(U1-VDD)
- C1 pad 2: Net-(IC2-VC2) -> B-
- C2 pad 1: B- -> Net-(U1-CDT)
- C2 pad 2: Net-(IC2-VC1) -> B-
- C3 pad 1: B- -> Net-(U2-VBATT)
- C3 pad 2: Net-(IC2-VDD) -> Net-(U2-CELL1)
- C8 pad 1: B- -> Net-(U2-REG2)
- C8 pad 2: Net-(IC2-CD) -> GND
- H1 pad 1: unconnected-(H1-Pad1) -> GND
- H2 pad 1: unconnected-(H2-Pad1) -> GND
- H3 pad 1: unconnected-(H3-Pad1) -> GND
- H4 pad 1: unconnected-(H4-Pad1) -> GND
- J11 pad 1: PACK+ -> +3V3
- J11 pad 2: B- -> +3V3
- J14 pad 1: VBATT -> PACK+
- J14 pad 2: VBATT -> PACK-
- J2 pad 2: PACK+_BF -> B+
- J4 pad 2: PACK+_BF -> B+
- J6 pad 2: PACK+_BF -> B+
- Q10 pad 1: Net-(Q10-G) -> Net-(U4-SENSE)
- Q10 pad 2: GND -> Net-(U4-SENSE)
- Q10 pad 3: Net-(Q10-D) -> Net-(U4-SENSE)
- Q11 pad 1: Net-(Q11-G) -> Net-(F2-Pad2)
- Q11 pad 2: GND -> Net-(F2-Pad2)
- Q11 pad 3: Net-(Q11-D) -> Net-(F2-Pad2)
- R18 pad 1: PACK+_BF -> B-
- R18 pad 2: Net-(IC2-VC2) -> Net-(U1-CTLC)
- R19 pad 1: BM -> B-
- R19 pad 2: Net-(IC2-VC1) -> Net-(U1-CTLD)
- R20 pad 1: BM -> Net-(U2-VBATT)
- R20 pad 2: Net-(R20-Pad2) -> B+
- R21 pad 1: Net-(R20-Pad2) -> Net-(U2-CELL1)
- R21 pad 2: Net-(IC2-VC1_CB) -> BM
- R22 pad 1: Net-(IC2-OUT) -> BM
- R22 pad 2: Net-(IC3-G) -> Net-(U1-VDD)
- R23 pad 1: Net-(IC2-VDD) -> Net-(U1-CO)
- R23 pad 2: PACK+_BF -> Net-(U3-CTLC)
- TH1 pad 1: BAT_THERM -> Net-(U2-AIN2)
- TP1 pad 1: B- -> B+
- TP10 pad 1: ENAB_BURN3 -> Net-(U2-AIN1)
- TP11 pad 1: ENAB_BURN4 -> Net-(Q10-G)
- TP12 pad 1: BAT_THERM -> Net-(Q11-G)
- TP4 pad 1: PACK+ -> Net-(U3-CTLC)
- TP5 pad 1: GND -> Net-(U3-CTLD)
- TP6 pad 1: VBATT -> PACK-
- TP7 pad 1: BURN_RELAY_A -> Net-(U2-AIN2)
- TP8 pad 1: ENAB_BURN1 -> /BatteryProtection/Alert_Fuel
- TP9 pad 1: ENAB_BURN2 -> Net-(U2-THRM)
Routing:
- net BAT_THERM: track 67.2 -> 0.00 mm, vias 1 -> 0
- net ENAB_BURN4: track 62.6 -> 0.00 mm, vias 2 -> 0
- net ENAB_BURN3: track 46.2 -> 0.00 mm, vias 2 -> 0
- net BURN_RELAY_A: track 40.9 -> 0.00 mm, vias 2 -> 0
- net B-: track 40.0 -> 0.00 mm, vias 19 -> 0
- net ENAB_BURN2: track 36.7 -> 0.00 mm, vias 2 -> 0
- net PACK+_BF: track 36.5 -> 0.00 mm, vias 34 -> 0
- net ENAB_BURN1: track 30.9 -> 0.00 mm, vias 2 -> 0
- net Net-(IC3-D): track 22.7 -> 0.00 mm, vias 2 -> 0
- net Net-(IC2-VC1): track 21.3 -> 0.00 mm
- net Net-(IC3-G): track 12.0 -> 0.00 mm, vias 2 -> 0
- net Net-(Q10-D): track 7.75 -> 0.00 mm
- net Net-(IC2-VC2): track 7.37 -> 0.00 mm
- net Net-(Q11-D): track 7.11 -> 0.00 mm
- net Net-(D2-A): track 6.98 -> 0.00 mm
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- removed copper zone on B.Cu, net /VBURN1
- removed copper zone on B.Cu, net /VBURN2
- removed copper zone on B.Cu, net /VBURN3
- removed copper zone on B.Cu, net /VBURN4
- removed copper zone on B.Cu, net /VBURN_A_IN
- removed copper zone on B.Cu, net B-
- removed copper zone on F.Cu, net B-
- removed copper zone on B.Cu, net BM
- removed copper zone on F.Cu, net BM
- removed copper zone on B.Cu, net GND
- removed copper zone on F.Cu, net GND
- removed copper zone on B.Cu, net PACK+
- removed copper zone on B.Cu, net PACK+_BF
- removed copper zone on F.Cu, net PACK+_BF
- removed copper zone on B.Cu, net VBATT
Other:
- copper layers 2 -> 4
- board text removed: "+"
- board text removed: "-"
- board text removed: "- +"
- board text removed: "7. 2 V"
- board text removed: "ARGUS - 1 BATTERY BOARD REV 2.0"
- board text removed: "B-"
- board text removed: "B2"
- board text removed: "B3"
- board text removed: "B4"
- board text removed: "BAT_THERM (OPTIONAL)"
- board text removed: "BM"
- board text removed: "BR"
- board text removed: "BT"
- board text removed: "GND"
- board text removed: "NTC Thermistor 10K - (103AT)"
- board text removed: "P+"
- board text removed: "P-"
- board text removed: "V+"

Commit message: Complete layout
Parts:
- removed J14: XT30PW, BatteryBoard:AMASS_XT30PW-M
- removed the J2 at (100.7, 62.7)
- removed the J4 at (100.7, 83.9)
- removed TP1, TP10, TP11, TP12, TP13, TP14, TP15, TP17, TP18, TP19, TP2, TP24, TP3, TP4, TP5, TP6, TP7, TP8, TP9: TestPoint, TestPoint:TestPoint_Loop_D1.80mm_Drill1.0mm_Beaded
- added F1: Polyfuse_Small, Resistor_SMD:R_1206_3216Metric, B.Cu at (173.2, 104.6)
- added F2: Polyfuse_Small, Resistor_SMD:R_1206_3216Metric, B.Cu at (175.5, 113.5)
- added J8: 282834-4, BatteryBoard:TE_282834-4, B.Cu at (186.6, 96.3)
- C1, C10, C11, C2, C6, C7, R18, R19, TH1, TH2, U4, U5: moved to B.Cu
- J1, J3: value Keystone-1042 -> Keystone-1048; footprint BatteryBoard:Keystone_1042 -> BatteryBoard:BAT_1048
- J2: renamed from J5; moved to B.Cu
- J7: renamed from J11; value 200528-0120 -> 200528-0100; footprint Connector_FFC-FPC:Molex_200528-0120_1x12-1MP_P1.00mm_Horizontal -> Connector_FFC-FPC:Molex_200528-0100_1x10-1MP_P1.00mm_Horizontal; moved to B.Cu
- Q1: renamed from Q10; moved to B.Cu
- Q2: renamed from Q12; moved to B.Cu
- Q3: renamed from Q11; moved to B.Cu
- Q4: renamed from Q13; moved to B.Cu
- R20: renamed from R22; moved to B.Cu
- R21: renamed from R23; moved to B.Cu
- R22: renamed from R24; moved to B.Cu
- R23: renamed from R26; moved to B.Cu
- R24: renamed from R30; moved to B.Cu
- R25: renamed from R29; moved to B.Cu
- U1: renamed from U3; moved to B.Cu
- U2: renamed from U1; moved to B.Cu
- moved H2 128.9 mm to (186.3, 139.2), turned to 90 degrees
- moved TH1 118.8 mm to (167.3, 69.1), turned to 90 degrees
- moved J7 116.3 mm to (107.6, 96.3), turned to 90 degrees
- moved H1 97.0 mm to (106.3, 139.2), turned to 90 degrees
- moved H3 88.9 mm to (186.3, 53.5), turned to -90 degrees
- moved TH2 87.5 mm to (167.3, 123.6), turned to -90 degrees
- moved J2 59.6 mm to (146.3, 66.6)
- moved J3 56.1 mm to (146.3, 116.5), turned to 0 degrees
- moved R17 52.7 mm to (169.8, 87.1), turned to -90 degrees
- moved R15 52.4 mm to (175.8, 93.5), turned to 180 degrees
- moved R16 51.1 mm to (171.2, 87.1), turned to -90 degrees
- moved C5 51.0 mm to (179.1, 92.0), turned to 0 degrees
- moved J4 50.3 mm to (146.3, 126.1), turned to 0 degrees
- moved C3 49.8 mm to (175.8, 92.0), turned to 180 degrees
- moved C4 49.4 mm to (175.8, 90.5), turned to 180 degrees
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- renumbered J6 to J4, Q15 to Q5, Q14 to Q6, Q17 to Q7, Q16 to Q8, R31 to R1, R40 to R10, R41 to R11, R42 to R12, R25 to R13, R20 to R14, R21 to R15, R27 to R16, R28 to R17, R32 to R2, R33 to R3, R34 to R4, R35 to R5, R36 to R6, R37 to R7, R38 to R8, R39 to R9, U2 to U3
Connections:
- J3 pad 1: B- -> BM
- J3 pad 2: BM -> B+
- J7 pad 1: +3V3 -> GND
- J7 pad 10: /Fuel_Alert -> +3V3
- J7 pad 2: +3V3 -> DSTAT
- J7 pad 3: +3V3 -> CSTAT
- J7 pad 4: GND -> ALRT
- J7 pad 5: GND -> SCL1
- J7 pad 6: /CHRG_STAT -> SDA1
- J7 pad 7: /DCHRG_STAT -> GND
- J7 pad 8: SCL1 -> GND
- J7 pad 9: SDA1 -> +3V3
- U3 pad 8: /BatteryProtection/Alert_Fuel -> ALRT
- U4 pad 4: /BatteryProtection/CHRG_STAT -> CSTAT
- U5 pad 4: /BatteryProtection/DCHRG_STAT -> DSTAT
Routing:
- net +3V3: track 0.00 -> 87.6 mm, vias 0 -> 8
- net CSTAT: track 0.00 -> 85.8 mm, vias 0 -> 2
- net DSTAT: track 0.00 -> 78.3 mm, vias 0 -> 2
- net ALRT: track 0.00 -> 70.2 mm, vias 0 -> 2
- net SCL1: track 0.00 -> 64.6 mm, vias 0 -> 2
- net SDA1: track 0.00 -> 60.0 mm, vias 0 -> 2
- net BM: track 0.00 -> 53.6 mm, vias 0 -> 105
- net Net-(U3-AIN1): track 0.00 -> 41.6 mm
- net SDA_Fuel: track 0.00 -> 30.1 mm, vias 0 -> 2
- net SCL_Fuel: track 0.00 -> 26.7 mm, vias 0 -> 2
- net Net-(Q3-G): track 0.00 -> 25.1 mm, vias 0 -> 2
- net Net-(U3-AIN2): track 0.00 -> 23.6 mm
- net Net-(U2-CO): track 0.00 -> 19.1 mm, vias 0 -> 2
- net Net-(U2-DO): track 0.00 -> 18.9 mm, vias 0 -> 2
- net Net-(Q1-G): track 0.00 -> 18.8 mm, vias 0 -> 2
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- added copper zone on B.Cu, net +3V3
- added copper zone on B.Cu, net B+
- added copper zone on F.Cu, net B+
- added copper zone on B.Cu, net B-
- added copper zone on F.Cu, net B-
- added copper zone on F.Cu, net BM
- added copper zone on B.Cu, net GND
- added copper zone on In1.Cu, net GND
- added copper zone on In2.Cu, net GND
- added copper zone on B.Cu, net Net-(F2-Pad2)
- added copper zone on B.Cu, net Net-(Q1-D)
- added copper zone on B.Cu, net Net-(Q3-D)
- added copper zone on B.Cu, net Net-(U4-SENSE)
- added copper zone on B.Cu, net PACK+
- added copper zone on B.Cu, net PACK-
Other:
- board size 95.9 x 90.2 mm -> 90.2 x 95.9 mm
- board text added: "+"
- board text added: "-"
- board text added: "1"
- board text added: "10"
- board text added: "3.3V"
- board text added: "ALRT"
- board text added: "ARGUS-1 Cubesat Carnegie Mellon University BatteryBoard v1 N. Khera M. Holliday"
- board text added: "CSTAT"
- board text added: "DSTAT"
- board text added: "GND"
- board text added: "MAINBOARD"
- board text added: "SCL"
- board text added: "SDA"
- board text added: "TR"

Commit message: Moved things idek
Parts:
- moved H4 3.81 mm to (110.1, 53.5)
- moved H3 2.54 mm to (183.8, 53.5)
Routing:
- added copper zone on B.Cu, net BM
Changed lines of the file:
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@@
 	(footprint "BatteryBoard:MountingHole"
 		(layer "F.Cu")
-		(at 186.309 53.4797 -90)
+		(at 183.769 53.4797 -90)
 		(descr "Mounting Hole 3.2mm, M3")
 		(tags "mounting hole 3.2mm m3")
@@
 	(footprint "BatteryBoard:MountingHole"
 		(layer "B.Cu")
-		(at 106.299 53.4797 90)
+		(at 110.109 53.4797 90)
 		(descr "Mounting Hole 3.2mm, M3")
 		(tags "mounting hole 3.2mm m3")
@@
 	)
 	(gr_text "TR"
-		(at 189.9158 53.4924 0)
+		(at 187.8584 53.4924 0)
 		(layer "F.SilkS")
 		(effects
@@
 		(start 167.259 89.31689)
 		(end 167.259 123.56084)
-		(width 0.635)
+		(width 0.508)
 		(layer "B.Cu")
 		(net 40)
@@
 		(start 168.65429 87.9216)
 		(end 167.259 89.31689)
-		(width 0.635)
+		(width 0.508)
 		(layer "B.Cu")
 		(net 40)
@@
 		(start 169.7625 87.9216)
 		(end 168.65429 87.9216)
-		(width 0.635)
+		(width 0.508)
 		(layer "B.Cu")
 		(net 40)
@@
 		(polygon
 			(pts
-				(xy 146.5707 96.0882) (xy 194.2465 96.0882) (xy 194.2465 59.0804) (xy 180.7083 59.0804) (xy 180.7083 47.9044)
+				(xy 146.5707 96.0882) (xy 194.2465 96.0882) (xy 194.2465 59.0804) (xy 178.1683 59.0804) (xy 178.1683 47.9044)
 				(xy 146.5707 47.9044)
 			)
@@
 			(pts
 				(xy 146.0373 145.4658) (xy 111.8997 145.4658) (xy 111.8997 133.604) (xy 98.3615 133.604) (xy 98.3615 59.0804)
-				(xy 111.8997 59.0804) (xy 111.8997 47.9044) (xy 146.0373 47.9044)
+				(xy 115.7097 59.0804) (xy 115.7097 47.9044) (xy 146.0373 47.9044)
 			)
 		)
@@
 			)
 		)
+	)
+	(zone
+		(net 2)
+		(net_name "BM")
+		(layer "B.Cu")
+		(hatch edge 0.5)
+		(priority 3)
+		(connect_pads yes
+			(clearance 0.254)
+		)
+		(min_thickness 0.254)
+		(filled_areas_thickness no)
+		(fill yes
+			(thermal_gap 0.5)
+			(thermal_bridge_width 0.5)
+			(island_removal_mode 1)
+			(island_area_min 9.999999)
+		)
+		(polygon
+			(pts
+				(xy 102.8954 63.3984) (xy 117.6528 63.3984) (xy 117.6528 69.8754) (xy 102.8954 69.8754)
+			)
+		)
+	)
+	(zone
+		(net 2)
+		(net_name "BM")
+		(layer "B.Cu")
+		(hatch edge 0.5)
+		(priority 3)
+		(connect_pads yes
+			(clearance 0.254)
+		)
+		(min_thickness 0.254)
+		(filled_areas_thickness no)
+		(fill yes
+			(thermal_gap 0.5)
+			(thermal_bridge_width 0.5)
+			(island_removal_mode 1)
+			(island_area_min 9.999999)
+		)
+		(polygon
+			(pts
+				(xy 102.8954 122.809) (xy 117.6528 122.809) (xy 117.6528 129.286) (xy 102.8954 129.286)
+			)
+		)

Commit message: v1 Final
Other:
- board text added: "INSTALL FIRST"
Changed lines of the file:
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@@
 			(usegerberextensions no)
 			(usegerberattributes yes)
-			(usegerberadvancedattributes no)
-			(creategerberjobfile no)
+			(usegerberadvancedattributes yes)
+			(creategerberjobfile yes)
 			(dashed_line_dash_ratio 12.000000)
 			(dashed_line_gap_ratio 3.000000)
@@
 			(drillshape 0)
 			(scaleselection 1)
-			(outputdirectory "gerbers/")
+			(outputdirectory "../../Gerbers/BatteryBoard")
 		)
 	)
@@
 		(at 146.304 66.63436 180)
 		(property "Reference" "J2"
-			(at 0 0 0)
+			(at 0.0254 8.29056 0)
 			(layer "B.SilkS")
 			(effects
@@
 		)
 	)
+	(gr_text "INSTALL FIRST"
+		(at 146.304 66.6242 -0)
+		(layer "B.SilkS")
+		(effects
+			(font
+				(size 0.889 0.889)
+				(thickness 0.127)
+			)
+			(justify mirror)
+		)
+	)
 	(gr_text "+"
 		(at 188.9506 100.1014 -90)
@@
 		)
 	)
+	(gr_text "INSTALL FIRST"
+		(at 146.304 86.3092 0)
+		(layer "F.SilkS")
+		(effects
+			(font
+				(size 0.889 0.889)
+				(thickness 0.127)
+			)
+		)
+	)
 	(gr_text "-"
 		(at 188.7474 92.4814 90)
@@
 		(layer "F.SilkS")
 		(effects
+			(font
+				(size 0.889 0.889)
+				(thickness 0.127)
+			)
+		)
+	)
+	(gr_text "INSTALL FIRST"
+		(at 146.304 66.6242 0)
+		(layer "F.SilkS")
+		(effects

Commit message: Relabeled I2C nets for accuracy
Connections:
- net SCL1 renamed SCL
- net SDA1 renamed SDA
Changed lines of the file:
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@@
 	(net 26 "Net-(Q5B-B2)")
 	(net 27 "Net-(Q5A-B1)")
-	(net 28 "SCL1")
+	(net 28 "SCL")
 	(net 29 "SCL_Fuel")
 	(net 30 "Net-(Q6A-G2)")
 	(net 31 "Net-(Q7A-B1)")
 	(net 32 "Net-(Q7B-B2)")
-	(net 33 "SDA1")
+	(net 33 "SDA")
 	(net 34 "Net-(Q8A-G2)")
 	(net 35 "SDA_Fuel")
@@
 			(layers "B.Cu" "B.Paste" "B.Mask")
 			(roundrect_rratio 0.25)
-			(net 33 "SDA1")
+			(net 33 "SDA")
 			(pinfunction "E1")
 			(pintype "passive")
@@
 			(layers "B.Cu" "B.Paste" "B.Mask")
 			(roundrect_rratio 0.25)
-			(net 33 "SDA1")
+			(net 33 "SDA")
 			(pinfunction "C2")
 			(pintype "passive")
@@
 			(layers "B.Cu" "B.Paste" "B.Mask")
 			(roundrect_rratio 0.25)
-			(net 33 "SDA1")
+			(net 33 "SDA")
 			(pintype "passive")
 		)
@@
 			(size 0.4 1)
 			(layers "B.Cu" "B.Paste" "B.Mask")
-			(net 28 "SCL1")
+			(net 28 "SCL")
 			(pinfunction "Pin_5")
 			(pintype "passive")
@@
 			(size 0.4 1)
 			(layers "B.Cu" "B.Paste" "B.Mask")
-			(net 33 "SDA1")
+			(net 33 "SDA")
 			(pinfunction "Pin_6")
 			(pintype "passive")
@@
 			(layers "B.Cu" "B.Paste" "B.Mask")
 			(roundrect_rratio 0.25)
-			(net 28 "SCL1")
+			(net 28 "SCL")
 			(pintype "passive")
 		)
@@
 			(layers "B.Cu" "B.Paste" "B.Mask")
 			(roundrect_rratio 0.25)
-			(net 28 "SCL1")
+			(net 28 "SCL")
 			(pinfunction "E1")
 			(pintype "passive")
@@
 			(layers "B.Cu" "B.Paste" "B.Mask")
 			(roundrect_rratio 0.25)
-			(net 28 "SCL1")
+			(net 28 "SCL")
 			(pinfunction "C2")
 			(pintype "passive")
